File: NRF52_IoT/NRF52_IoT.kicad_sch (KiCad schematic)
At the start: 1 part, among them U1 nRF52840

Commit message: Update NRF52_IoT.kicad_sch
Parts:
- U1: MOUSER (none) -> https://ro.mouser.com/ProductDetail/Nordic-Semiconductor/nR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
Connections:
- net GND: now reaches U1.B7 (VSS), U1.EP (VSS)
- net GND: now also U1.F23 (VSS_PA)
Other:
- moved on the sheet: U1
Changed lines of the file:
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@@
 (kicad_sch (version 20211123) (generator eeschema)
   (paper "A4")
-  (symbol (lib_id "MCU_Nordic:nRF52840") (at 81.28 99.06 0) (unit 1)
+  (junction (at 73.66 182.88) (diameter 0) (color 0 0 0 0)
+  )
+  (wire (pts (xy 76.2 182.88) (xy 76.2 180.34))
+    (stroke (width 0) (type default) (color 0 0 0 0))
+  )
+  (wire (pts (xy 73.66 182.88) (xy 73.66 185.42))
+    (stroke (width 0) (type default) (color 0 0 0 0))
+  )
+  (wire (pts (xy 73.66 180.34) (xy 73.66 182.88))
+    (stroke (width 0) (type default) (color 0 0 0 0))
+  )
+  (wire (pts (xy 73.66 182.88) (xy 76.2 182.88))
+    (stroke (width 0) (type default) (color 0 0 0 0))
+  )
+  (symbol (lib_id "power:GND") (at 73.66 185.42 0) (unit 1)
     (in_bom yes) (on_board yes) (fields_autoplaced)
-    (property "Reference" "U1" (id 0) (at 85.8394 167.64 0)
+    (property "Reference" "#PWR?" (id 0) (at 73.66 191.77 0)
+      (effects (font (size 1.27 1.27)) hide)
+    )
+    (property "Value" "GND" (id 1) (at 73.66 190.5 0)
+      (effects (font (size 1.27 1.27)) hide)
+    )
+    (property "Footprint" "" (id 2) (at 73.66 185.42 0)
+      (effects (font (size 1.27 1.27)) hide)
+    )
+    (property "Datasheet" "" (id 3) (at 73.66 185.42 0)
+      (effects (font (size 1.27 1.27)) hide)
+    )
+    (pin "1")
+  )
+  (symbol (lib_id "MCU_Nordic:nRF52840") (at 73.66 109.22 0) (unit 1)
+    (in_bom yes) (on_board yes) (fields_autoplaced)
+    (property "Reference" "U1" (id 0) (at 78.2194 177.8 0)
       (effects (font (size 1.27 1.27)) (justify left))
     )
-    (property "Value" "nRF52840" (id 1) (at 85.8394 170.18 0)
+    (property "Value" "nRF52840" (id 1) (at 78.2194 180.34 0)
       (effects (font (size 1.27 1.27)) (justify left))
     )
-    (property "Footprint" "Package_DFN_QFN:Nordic_AQFN-73-1EP_7x7mm_P0.5mm" (id 2) (at 81.28 172.72 0)
+    (property "Footprint" "Package_DFN_QFN:Nordic_AQFN-73-1EP_7x7mm_P0.5mm" (id 2) (at 73.66 182.88 0)
       (effects (font (size 1.27 1.27)) hide)
     )
-    (property "Datasheet" "http://infocenter.nordicsemi.com/topic/com.nordic.infocenter.nrf52/dita/nrf52/chips/nrf52840.html" (id 3) (at 64.77 50.8 0)
+    (property "Datasheet" "http://infocenter.nordicsemi.com/topic/com.nordic.infocenter.nrf52/dita/nrf52/chips/nrf52840.html" (id 3) (at 57.15 60.96 0)
+      (effects (font (size 1.27 1.27)) hide)
+    )
+    (property "MOUSER" "https://ro.mouser.com/ProductDetail/Nordic-Semiconductor/nRF52840-QIAA-T?qs=AQlKX63v8RtTyx08F8csPQ%3D%3D" (id 4) (at 73.66 109.22 0)
       (effects (font (size 1.27 1.27)) hide)
     )
@@
   )
   (symbol_instances
+    (path "/78a63942-3622-4f97-b069-b1943a504400"
+      (reference "#PWR?") (unit 1) (value "GND") (footprint "")
+    )
     (path "/e3c62471-d367-4c95-8294-c8f55f87ab86"
       (reference "U1") (unit 1) (value "nRF52840") (footprint "Package_DFN_QFN:Nordic_AQFN-73-1EP_7x7mm_P0.5mm")
